Commit message: use latest urdf file

File: share/urdf/nao_robot.urdf (robot description, URDF)
Before this commit: robot naoH25V50, 77 links, 76 joints
Links:
- added link CameraBottom_optical_frame
- added link CameraTop_optical_frame
Joints:
- added joint CameraBottom_optical_frame_joint: type fixed, parent CameraBottom_frame, child CameraBottom_optical_frame, origin xyz=0 0 0 rpy=-1.57079632679 0 -1.57079632679
- added joint CameraTop_optical_frame_joint: type fixed, parent CameraTop_frame, child CameraTop_optical_frame, origin xyz=0 0 0 rpy=-1.57079632679 0 -1.57079632679
- joint Sonar/Left_sensor_fixedjoint: child RSonar_frame -> LSonar_frame
- joint Sonar/Right_sensor_fixedjoint: child LSonar_frame -> RSonar_frame
