Commit message: add optical frame

File: share/urdf/pepper.urdf (robot description, URDF)
Before this commit: robot julietteY20MP, 78 links, 77 joints
Links:
- added link CameraBottom_optical_frame
- added link CameraDepth_optical_frame
- added link CameraTop_optical_frame
Joints:
- added joint CameraBottom_optical_frame_joint: type fixed, parent CameraBottom_frame, child CameraBottom_optical_frame, origin xyz=0 0 0 rpy=-1.57079632679 0 -1.57079632679
- added joint CameraDepth_optical_frame_joint: type fixed, parent CameraDepth_frame, child CameraDepth_optical_frame, origin xyz=0 0 0 rpy=-1.57079632679 0 -1.57079632679
- added joint CameraTop_optical_frame_joint: type fixed, parent CameraTop_frame, child CameraTop_optical_frame, origin xyz=0 0 0 rpy=-1.57079632679 0 -1.57079632679
- joint Head/Touch/Front_sensor_fixedjoint: origin xyz=0.0275 0 0.1245 rpy=0 -1.1861 0 -> xyz=0.028175 0 0.21267 rpy=0 0.20944 0
- joint Head/Touch/Middle_sensor_fixedjoint: origin xyz=-0.004 0 0.125 rpy=3.14159 -1.57079 -3.14159 -> xyz=0.0041 0 0.2159 rpy=0 -0.0349066 0
- joint Head/Touch/Rear_sensor_fixedjoint: origin xyz=-0.033 0 0.1245 rpy=3.14159 -1.33319 -3.14159 -> xyz=-0.03376 0 0.21052 rpy=0 -0.314159 0
- joint LaserSensor/Front_sensor_fixedjoint: origin xyz=0.0562 0 -0.0692 rpy=0 0.349044 0 -> xyz=0.0562 0 -0.334 rpy=0 0 0
- joint LaserSensor/Left_sensor_fixedjoint: origin xyz=-0.018 0.0899 -0.0759 rpy=8.34035e-09 0.191982 1.5708 -> xyz=-0.018 0.0899 -0.334 rpy=0 0 1.75728367321
- joint LaserSensor/Right_sensor_fixedjoint: origin xyz=0.018 -0.0899 -0.0759 rpy=4.08851e-07 0.191857 -1.60746 -> xyz=-0.018 -0.0899 -0.334 rpy=0 0 -1.75728367321

Commit message: update the Pepper URDF

File: share/urdf/pepper.urdf (robot description, URDF)
Before this commit: robot julietteY20MP, 81 links, 80 joints
Links:
- added link SurroundingFrontLaser_device_frame
- added link SurroundingLeftLaser_device_frame
- added link SurroundingRightLaser_device_frame
- link LFinger11_link: mass None -> 2e-06
- link LFinger12_link: mass None -> 2e-06
- link LFinger13_link: mass None -> 2e-06
- link LFinger21_link: mass None -> 2e-06
- link LFinger22_link: mass None -> 2e-06
- link LFinger23_link: mass None -> 2e-06
- link LFinger31_link: mass None -> 2e-06
- link LFinger32_link: mass None -> 2e-06
- link LFinger33_link: mass None -> 2e-06
- link LFinger41_link: mass None -> 2e-06
- link LFinger42_link: mass None -> 2e-06
- link LFinger43_link: mass None -> 2e-06
- link LThumb1_link: mass None -> 2e-06
- link LThumb2_link: mass None -> 2e-06
- link RFinger11_link: mass None -> 2e-06
- link RFinger12_link: mass None -> 2e-06
- link RFinger13_link: mass None -> 2e-06
- link RFinger21_link: mass None -> 2e-06
- link RFinger22_link: mass None -> 2e-06
- link RFinger23_link: mass None -> 2e-06
- link RFinger31_link: mass None -> 2e-06
- link RFinger32_link: mass None -> 2e-06
- link RFinger33_link: mass None -> 2e-06
- link RFinger41_link: mass None -> 2e-06
- link RFinger42_link: mass None -> 2e-06
- link RFinger43_link: mass None -> 2e-06
- link RThumb1_link: mass None -> 2e-06
- link RThumb2_link: mass None -> 2e-06
- link l_gripper: mass None -> 2e-06
- link r_gripper: mass None -> 2e-06
Joints:
- removed joint CameraBottom_optical_frame_joint
- removed joint CameraDepth_optical_frame_joint
- removed joint CameraTop_optical_frame_joint
- added joint CameraBottom_optical_frame_fixedjoint: type fixed, parent CameraBottom_frame, child CameraBottom_optical_frame, origin xyz=0 0 0 rpy=-1.57079632679 0 -1.57079632679
- added joint CameraDepth_optical_frame_fixedjoint: type fixed, parent CameraDepth_frame, child CameraDepth_optical_frame, origin xyz=0 0 0 rpy=-1.57079632679 0 -1.57079632679
- added joint CameraTop_optical_frame_fixedjoint: type fixed, parent CameraTop_frame, child CameraTop_optical_frame, origin xyz=0 0 0 rpy=-1.57079632679 0 -1.57079632679
- added joint LaserSensor/Front_projected_sensor_fixedjoint: type fixed, parent Tibia, child SurroundingFrontLaser_frame, origin xyz=0.0562 0 -0.334 rpy=0 0 0, axis 0 0 0
- added joint LaserSensor/Left_projected_sensor_fixedjoint: type fixed, parent Tibia, child SurroundingLeftLaser_frame, origin xyz=-0.018 0.0899 -0.334 rpy=0 0 1.75728, axis 0 0 0
- added joint LaserSensor/Right_projected_sensor_fixedjoint: type fixed, parent Tibia, child SurroundingRightLaser_frame, origin xyz=-0.018 -0.0899 -0.334 rpy=0 0 -1.75728, axis 0 0 0
- joint LaserSensor/Front_sensor_fixedjoint: child SurroundingFrontLaser_frame -> SurroundingFrontLaser_device_frame; origin xyz=0.0562 0 -0.334 rpy=0 0 0 -> xyz=0.0562 0 -0.0692 rpy=0 0.349044 0
- joint LaserSensor/Left_sensor_fixedjoint: child SurroundingLeftLaser_frame -> SurroundingLeftLaser_device_frame; origin xyz=-0.018 0.0899 -0.334 rpy=0 0 1.75728367321 -> xyz=-0.018 0.0899 -0.0759 rpy=8.34035e-09 0.191982 1.5708
- joint LaserSensor/Right_sensor_fixedjoint: child SurroundingRightLaser_frame -> SurroundingRightLaser_device_frame; origin xyz=-0.018 -0.0899 -0.334 rpy=0 0 -1.75728367321 -> xyz=-0.018 -0.0899 -0.0759 rpy=4.08851e-07 0.191857 -1.60746

Commit message: Edit urdf for the external URG

File: share/urdf/pepper.urdf (robot description, URDF)
Before this commit: robot JulietteY20MP, 84 links, 83 joints
Links:
- added link ExternalLaser_frame
Joints:
- added joint LaserSensor/External_sensor_fixedjoint: type fixed, parent Tibia, child ExternalLaser_frame, origin xyz=0.1579 0 -0.1073 rpy=0 0 0, axis 0 0 0
